File: lifi elec/lifi.kicad_sch (KiCad schematic)
At the start: 14 parts, among them J1 Raspberry_Pi, Q1 Phototransistor, Q2 Phototransistor, Q3 2N2222, U1 AO

Commit message: small update
Parts:
- added J2: Raspberry_Pi, symbol Connector:Raspberry_Pi_2_3
- added R2, R6: R, symbol Device:R
- added base: R_Photo, OptoDevice:R_LDR_4.9x4.2mm_P2.54mm_Vertical, symbol Device:R_Photo
- added photo: R_Photo, symbol Device:R_Photo
Connections:
- new net: J2.1 (3V3), J2.17 (3V3), base.1, photo.1
- new net: J2.13 (GPIO27), R6.2, base.2
- new net: J2.14 (GND), J2.20 (GND), J2.25 (GND), J2.30 (GND), J2.34 (GND), J2.39 (GND), J2.6 (GND), J2.9 (GND), R2.2, R6.1
- new net: J2.2 (5V), J2.4 (5V)
- new net: J2.37 (GPIO26), R2.1, photo.2

Commit message: updating schematics
Parts:
- removed D1, D2: LED, symbol Device:LED
- removed MES1, MES2: Oscilloscope, symbol Device:Oscilloscope
- removed Q1, Q2: Phototransistor, LED_THT:LED_D5.0mm_Clear, symbol Sensor_Optical:BPW40
- removed R4: 100, symbol Device:R
- removed R5: 1000, symbol Device:R
- removed U1: AO, Package_SO:SOIC-8-1EP_3.9x4.9mm_P1.27mm_EP2.29x3mm, symbol Amplifier_Operational:ADA4625-2ARDZ
- added J3: Raspberry_Pi, symbol Connector:Raspberry_Pi_2_3
- added base, photo: Phototransistor, OptoDevice:Osram_LPT80A, symbol Sensor_Optical:LPT80A
- Q3: value 2N2222 -> Transistor
- R3: value 230 -> R
Connections:
- net at R1.2: now also R3.1, J3.14 (GND), J3.20 (GND), J3.25 (GND), J3.30 (GND), J3.34 (GND), J3.39 (GND), J3.6 (GND), J3.9 (GND)
- net at D3.1 (K): now also Q3.3 (C); no longer Q3.1 (E)
- net at J1.14 (GND), J1.20 (GND), J1.25 (GND)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: now also Q3.1 (E); no longer Q3.3 (C)
- net at R3.2: now also J3.13 (GPIO27), base.2 (E)
- net AC: no longer names the net of R1.1
- net AC: now also J3.37 (GPIO26), photo.2 (E); no longer R3.1
- new net: J3.1 (3V3), J3.17 (3V3), base.1 (C), photo.1 (C)
- new net: J3.2 (5V), J3.4 (5V)
Other:
- moved on the sheet: base, photo
